Commit message: wip-16.09.2020

File: src/abot_description/urdf/sensors.xacro (robot description, xacro)
@@ -25,5 +25,5 @@
 	<!-- Lidar joint -->
 	<joint name="laser_link_to_base" type="fixed">
-		<origin xyz="0.022 0 0.18315" rpy="0 0 0" />
+		<origin xyz="0.022 0 0.18315" rpy="0 0 ${PI}" />
 		<parent link="abot_base" />
 		<child link="laser_link" />
