Commit message: wip-15.09.2020

File: src/abot_description/urdf/abot.xacro (robot description, xacro)
@@ -1,4 +1,5 @@
 <?xml version="1.0"?>
-<robot name="abot" xmlns:xacro="http://www.ros.org/wiki/xacro">
+<robot name="abot"
+	xmlns:xacro="http://www.ros.org/wiki/xacro">
 	<!-- Macro -->
 	<xacro:include filename="$(find abot_description)/urdf/macros.xacro" />
@@ -11,5 +12,5 @@
 	<xacro:property name="wheel_width" value="0.0158" />
 	<xacro:property name="wheel_separation" value="0.128" />
-	<xacro:property name="clearance" value="0.01795" />
+	<xacro:property name="clearance" value="0.01745" />
 	<xacro:property name="wheel_mass" value="0.032704" />
 	<xacro:property name="caster_wheel_mass" value="0.011207" />
@@ -48,7 +49,7 @@
 	<link name="abot_base">
 		<inertial>
-			<origin xyz="-0.0153999844033198 8.13067891968615E-15 0.0121543976022896" rpy="0 0 0" />
-			<mass value="0.469829440847482" />
-			<inertia ixx="0.000570631411959662" ixy="2.91510421236034E-09" ixz="-2.38329846370416E-05" iyy="0.000513725189549573" iyz="1.47383106149314E-09" izz="0.000868674371165525" />
+			<origin xyz="-0.0127093410022275 -1.41221243673916E-07 0.039639861536933" rpy="0 0 0" />
+			<mass value="0.833887267376891" />
+			<inertia ixx="0.00120589522768881" ixy="6.98274532230061E-09" ixz="-2.38252631510239E-05" iyy="0.00114896877416948" iyz="1.47383105573365E-09" izz="0.00213840106572274" />
 		</inertial>
 		<visual>
@@ -70,3 +71,5 @@
 	<xacro:include filename="$(find abot_description)/urdf/right_wheel.xacro" />
 	<xacro:include filename="$(find abot_description)/urdf/caster_wheel.xacro" />
+	<!-- Sensors -->
+	<xacro:include filename="$(find abot_description)/urdf/sensors.xacro" />
 </robot>

File: src/abot_description/urdf/caster_wheel.xacro (robot description, xacro)
@@ -46,5 +46,5 @@
 	<!-- caster wheel joints -->
 	<joint name="caster_wheel_to_base" type="fixed">
-		<origin xyz="-0.078 0 -0.01095" rpy="0 0 0" />
+		<origin xyz="-0.0780000000000001 0 -0.0104499999999992" rpy="0 0 0" />
 		<parent link="abot_base" />
 		<child link="caster_wheel" />

File: src/abot_description/urdf/left_wheel.xacro (robot description, xacro)
@@ -46,5 +46,5 @@
 	<!-- Left wheel joints -->
 	<joint name="left_wheel_to_base" type="continuous">
-		<origin xyz="0 0.064 0.014" rpy="0 0 0" />
+		<origin xyz="0 0.0639999999999998 0.0145000000000007" rpy="0 0 0" />
 		<parent link="abot_base" />
 		<child link="left_wheel" />

File: src/abot_description/urdf/right_wheel.xacro (robot description, xacro)
@@ -46,5 +46,5 @@
 	<!-- Right wheel joints -->
 	<joint name="right_wheel_to_base" type="continuous">
-		<origin xyz="0 -0.064 0.014" rpy="0 0 0" />
+		<origin xyz="0 -0.0640000000000002 0.0144999999999993" rpy="0 0 0" />
 		<parent link="abot_base" />
 		<child link="right_wheel" />

Commit message: wip-22.09.2020

File: src/abot_description/urdf/abot.xacro (robot description, xacro)
@@ -49,7 +49,7 @@
 	<link name="abot_base">
 		<inertial>
-			<origin xyz="-0.0127093410022275 -1.41221243673916E-07 0.039639861536933" rpy="0 0 0" />
-			<mass value="0.833887267376891" />
-			<inertia ixx="0.00120589522768881" ixy="6.98274532230061E-09" ixz="-2.38252631510239E-05" iyy="0.00114896877416948" iyz="1.47383105573365E-09" izz="0.00213840106572274" />
+			<origin xyz="-0.013369146216312 -2.32945596953608E-07 0.0424852261575198" rpy="0 0 0" />
+			<mass value="0.505536908309907" />
+			<inertia ixx="0.000583839286669347" ixy="6.98274532231354E-09" ixz="-8.88829560312885E-06" iyy="0.000559099682201411" iyz="1.47383106096032E-09" izz="0.00104254331700213" />
 		</inertial>
 		<visual>

File: src/abot_description/urdf/matherials.xacro (robot description, xacro)
@@ -13,3 +13,6 @@
 		<color rgba="1.0 1.0 1.0 1.0"/>
 	</material>
+	<material name="Yellow">
+		<color rgba="1.0 1.0 0.0 1.0"/>
+	</material>
 </robot>

File: src/abot_description/urdf/sensors.xacro (robot description, xacro)
@@ -10,12 +10,12 @@
 		</inertial>
 		<visual>
-			<origin xyz="0 0 0" rpy="0 0 0" />
+			<origin xyz="0 0 0" rpy="0 0 ${PI}" />
 			<geometry>
 				<mesh filename="package://abot_description/meshes/laser_link.STL" />
 			</geometry>
-			<material name="Blue" />
+			<material name="Yellow" />
 		</visual>
 		<collision>
-			<origin xyz="0 0 0" rpy="0 0 0" />
+			<origin xyz="0 0 0" rpy="0 0 ${PI}" />
 			<geometry>
 				<mesh filename="package://abot_description/meshes/laser_link.STL" />
@@ -30,3 +30,87 @@
 		<axis xyz="0 0 0" />
 	</joint>
+	<!-- IR sensor front middle CAD link -->
+	<link name="ir_fm">
+		<inertial>
+			<origin xyz="-0.0193778284817564 0.0517927266118569 0.000510012680068063" rpy="0 0 0" />
+			<mass value="0.0029706780872837" />
+			<inertia ixx="2.75251627428986E-07" ixy="9.10709415904095E-08" ixz="-7.93160400909887E-10" iyy="1.17636929894439E-07" iyz="8.3896081509796E-11" izz="2.95301311766455E-07" />
+		</inertial>
+		<visual>
+			<origin xyz="0 0 0" rpy="0 0 0" />
+			<geometry>
+				<mesh filename="package://abot_description/meshes/ir_fm.STL" />
+			</geometry>
+			<material name="Yellow" />
+		</visual>
+		<collision>
+			<origin xyz="0 0 0" rpy="0 0 0" />
+			<geometry>
+				<mesh filename="package://abot_description/meshes/ir_fm.STL" />
+			</geometry>
+		</collision>
+	</link>
+	<!-- IR sensor front middle joint -->
+	<joint name="ir_fm_to_base" type="fixed">
+		<origin xyz="0.0812 0 -0.0065" rpy="0 0 0" />
+		<parent link="abot_base" />
+		<child link="ir_fm" />
+		<axis xyz="0 0 0" />
+	</joint>
+	<!-- IR sensor front left CAD link -->
+	<link name="ir_fl">
+		<inertial>
+			<origin xyz="-0.00737194484411242 0.000279264844105703 0.000510014496335439" rpy="0 0 0" />
+			<mass value="0.00297067826138337" />
+			<inertia ixx="3.16734695808955E-07" ixy="-5.89288167867935E-09" ixz="-6.76347714169545E-10" iyy="7.61538286810033E-08" iyz="4.22675785570517E-10" izz="2.95301261269084E-07" />
+		</inertial>
+		<visual>
+			<origin xyz="0 0 0" rpy="0 0 0" />
+			<geometry>
+				<mesh filename="package://abot_description/meshes/ir_fl.STL" />
+			</geometry>
+			<material name="Yellow" />
+		</visual>
+		<collision>
+			<origin xyz="0 0 0" rpy="0 0 0" />
+			<geometry>
+				<mesh filename="package://abot_description/meshes/ir_fl.STL" />
+			</geometry>
+		</collision>
+	</link>
+	<!-- IR sensor front left joint -->
+	<joint name="ir_fl_to_base" type="fixed">
+		<origin xyz="0.068572 0.054769 -0.0065" rpy="0 0 0.45321" />
+		<parent link="abot_base" />
+		<child link="ir_fl" />
+		<axis xyz="0 0 0" />
+	</joint>
+	<!-- IR sensor front right CAD link -->
+	<link name="ir_fr">
+		<inertial>
+			<origin xyz="-0.0073719435479474 0.000279266429044269 0.000510012687927432" rpy="0 0 0" />
+			<mass value="0.00297067925092848" />
+			<inertia ixx="3.16734825741921E-07" ixy="-5.89285028889523E-09" ixz="-6.76367534098839E-10" iyy="7.61538418054215E-08" iyz="4.2267880693731E-10" izz="2.95301389790314E-07" />
+		</inertial>
+		<visual>
+			<origin xyz="0 0 0" rpy="0 0 0" />
+			<geometry>
+				<mesh filename="package://abot_description/meshes/ir_fr.STL" />
+			</geometry>
+			<material name="Yellow" />
+		</visual>
+		<collision>
+			<origin xyz="0 0 0" rpy="0 0 0" />
+			<geometry>
+				<mesh filename="package://abot_description/meshes/ir_fr.STL" />
+			</geometry>
+		</collision>
+	</link>
+	<!-- IR sensor front right joint -->
+	<joint name="ir_fr_to_base" type="fixed">
+		<origin xyz="0.0685721788194783 -0.0547694638499224 -0.00650000000000129" rpy="0 0 -0.45320639368436" />
+		<parent link="abot_base" />
+		<child link="ir_fr" />
+		<axis xyz="0 0 0" />
+	</joint>
 </robot>

Commit message: wip-06.10.2020

File: src/abot_description/urdf/abot.xacro (robot description, xacro)
@@ -10,8 +10,8 @@
 	<xacro:property name="wheel_radius" value="0.03195" />
 	<xacro:property name="caster_wheel_radius" value="0.007" />
-	<xacro:property name="wheel_width" value="0.0158" />
+	<xacro:property name="wheel_width" value="0.026" />
 	<xacro:property name="wheel_separation" value="0.128" />
-	<xacro:property name="clearance" value="0.01745" />
-	<xacro:property name="wheel_mass" value="0.032704" />
+	<xacro:property name="clearance" value="0.018" />
+	<xacro:property name="wheel_mass" value="0.050464" />
 	<xacro:property name="caster_wheel_mass" value="0.011207" />
 	<!-- Base_footprint -->
@@ -20,5 +20,5 @@
 			<origin xyz="0 0 0" rpy="0 0 0" />
 			<geometry>
-				<cylinder length="0.001" radius="0.100" />
+				<cylinder length="0.001" radius="0.010" />
 			</geometry>
 			<material name="Blue" />
@@ -49,7 +49,7 @@
 	<link name="abot_base">
 		<inertial>
-			<origin xyz="-0.013369146216312 -2.32945596953608E-07 0.0424852261575198" rpy="0 0 0" />
-			<mass value="0.505536908309907" />
-			<inertia ixx="0.000583839286669347" ixy="6.98274532231354E-09" ixz="-8.88829560312885E-06" iyy="0.000559099682201411" iyz="1.47383106096032E-09" izz="0.00104254331700213" />
+			<origin xyz="-0.0198506551333707 -2.90632176868541E-07 0.0455751019105062" rpy="0 0 0" />
+			<mass value="0.405194628185875" />
+			<inertia ixx="0.000555716898847813" ixy="4.06361886095622E-09" ixz="-9.13022146244237E-06" iyy="0.000532480608869663" iyz="-7.85503541476441E-11" izz="0.00101776419338989" />
 		</inertial>
 		<visual>

File: src/abot_description/urdf/caster_wheel.xacro (robot description, xacro)
@@ -5,7 +5,7 @@
 	<link name="caster_wheel1">
 		<inertial>
-			<origin xyz="1.3878E-17 3.4074E-19 -5.2042E-18" rpy="0 0 0" />
+			<origin xyz="0 1.6073E-19 0" rpy="0 0 0" />
 			<mass value="0.011207" />
-			<inertia ixx="2.1965E-07" ixy="9.9033E-38" ixz="6.4182E-38" iyy="2.1965E-07" iyz="-3.2108E-37" izz="2.1965E-07" />
+			<inertia ixx="2.1965E-07" ixy="9.9033E-38" ixz="1.9255E-37" iyy="2.1965E-07" iyz="-3.2209E-37" izz="2.1965E-07" />
 		</inertial>
 		<visual>
@@ -26,5 +26,5 @@
 	<link name="caster_wheel">
 		<inertial>
-			<origin xyz="1.3878E-17 3.4074E-19 -5.2042E-18" rpy="0 0 0" />
+			<origin xyz="0 1.6073E-19 0" rpy="0 0 0" />
 			<mass value="0.011207" />
 			<xacro:sphere_inertia mass="${caster_wheel_mass}" radius="${caster_wheel_radius}" />
@@ -46,5 +46,5 @@
 	<!-- caster wheel joints -->
 	<joint name="caster_wheel_to_base" type="fixed">
-		<origin xyz="-0.0780000000000001 0 -0.0104499999999992" rpy="0 0 0" />
+		<origin xyz="-0.0780000000000001 0 -0.0109999999999992" rpy="0 0 0" />
 		<parent link="abot_base" />
 		<child link="caster_wheel" />

File: src/abot_description/urdf/left_wheel.xacro (robot description, xacro)
@@ -5,7 +5,7 @@
 	<link name="left_wheel1">
 		<inertial>
-			<origin xyz="7.0481E-20 -0.00013293 0" rpy="0 0 0" />
+			<origin xyz="-1.7545E-10 0.00056576 6.1245E-11" rpy="0 0 0" />
 			<mass value="${wheel_mass}" />
-			<inertia ixx="1.034E-05" ixy="6.5778E-20" ixz="-1.1387E-12" iyy="1.9808E-05" iyz="9.9943E-20" izz="1.034E-05" />
+			<inertia ixx="2.0701E-05" ixy="3.2217E-14" ixz="8.6674E-12" iyy="3.5827E-05" iyz="3.3202E-15" izz="2.0701E-05" />
 		</inertial>
 		<visual>
@@ -26,5 +26,5 @@
 	<link name="left_wheel">
 		<inertial>
-			<origin xyz="7.0481E-20 -0.00013293 0" rpy="0 0 0" />
+			<origin xyz="-1.7545E-10 0.00056576 6.1245E-11" rpy="0 0 0" />
 			<mass value="${wheel_mass}" />
 			<xacro:cylinder_inertia mass="${wheel_mass}" radius="${wheel_radius}" height="${wheel_width}" />
@@ -46,8 +46,8 @@
 	<!-- Left wheel joints -->
 	<joint name="left_wheel_to_base" type="continuous">
-		<origin xyz="0 0.0639999999999998 0.0145000000000007" rpy="0 0 0" />
+		<origin xyz="0 0.0679999999999999 0.0145000000000007" rpy="0 0 0" />
 		<parent link="abot_base" />
 		<child link="left_wheel" />
-		<axis xyz="0 -1 0" />
+		<axis xyz="0 1 0" />
 	</joint>
 	<joint name="left_wheel_to_wheel1" type="fixed">

File: src/abot_description/urdf/right_wheel.xacro (robot description, xacro)
@@ -5,7 +5,7 @@
 	<link name="right_wheel1">
 		<inertial>
-			<origin xyz="2.6037E-18 0.00013293 5.2042E-18" rpy="0 0 0" />
+			<origin xyz="-1.1135E-10 -0.00056576 1.5533E-10" rpy="0 0 0" />
 			<mass value="${wheel_mass}" />
-			<inertia ixx="1.034E-05" ixy="6.5763E-20" ixz="-6.4107E-11" iyy="1.9808E-05" iyz="1.0024E-19" izz="1.034E-05" />
+			<inertia ixx="2.0701E-05" ixy="-6.0753E-15" ixz="6.4131E-11" iyy="3.5827E-05" iyz="3.275E-14" izz="2.0701E-05" />
 		</inertial>
 		<visual>
@@ -26,5 +26,5 @@
 	<link name="right_wheel">
 		<inertial>
-			<origin xyz="2.6037E-18 0.00013293 5.2042E-18" rpy="0 0 0" />
+			<origin xyz="-1.1135E-10 -0.00056576 1.5533E-10" rpy="0 0 0" />
 			<mass value="${wheel_mass}" />
 			<xacro:cylinder_inertia mass="${wheel_mass}" radius="${wheel_radius}" height="${wheel_width}" />
@@ -46,8 +46,8 @@
 	<!-- Right wheel joints -->
 	<joint name="right_wheel_to_base" type="continuous">
-		<origin xyz="0 -0.0640000000000002 0.0144999999999993" rpy="0 0 0" />
+		<origin xyz="0 -0.0680000000000002 0.0144999999999993" rpy="0 0 0" />
 		<parent link="abot_base" />
 		<child link="right_wheel" />
-		<axis xyz="0 1 0" />
+		<axis xyz="0 -1 0" />
 	</joint>
 	<joint name="right_wheel_to_wheel1" type="fixed">

File: src/abot_description/urdf/sensors.xacro (robot description, xacro)
@@ -25,43 +25,211 @@
 	<!-- Lidar joint -->
 	<joint name="laser_link_to_base" type="fixed">
-		<origin xyz="0.022 0 0.18315" rpy="0 0 ${PI}" />
+		<origin xyz="0.0219999999999071 0 0.178150000000001" rpy="0 0 ${PI}" />
 		<parent link="abot_base" />
 		<child link="laser_link" />
 		<axis xyz="0 0 0" />
 	</joint>
-	<!-- IR sensor front middle CAD link -->
+	<!-- IR sensor front CAD link -->
 	<link name="ir_f">
 		<inertial>
-			<origin xyz="-0.0193778284817564 0.0517927266118569 0.000510012680068063" rpy="0 0 0" />
-			<mass value="0.0029706780872837" />
-			<inertia ixx="2.75251627428986E-07" ixy="9.10709415904095E-08" ixz="-7.93160400909887E-10" iyy="1.17636929894439E-07" iyz="8.3896081509796E-11" izz="2.95301311766455E-07" />
-		</inertial>
-		<visual>
-			<origin xyz="0 0 0" rpy="0 0 0" />
-			<geometry>
-				<mesh filename="package://abot_description/meshes/ir_fm.STL" />
-			</geometry>
-			<material name="Yellow" />
-		</visual>
-		<collision>
-			<origin xyz="0 0 0" rpy="0 0 0" />
-			<geometry>
-				<mesh filename="package://abot_description/meshes/ir_fm.STL" />
-			</geometry>
-		</collision>
-	</link>
-	<!-- IR sensor front middle joint -->
+			<origin xyz="-0.0073719 -0.00051001 0.00027926" rpy="0 0 0" />
+			<mass value="0.0029707" />
+			<inertia ixx="3.1673E-07" ixy="6.7636E-10" ixz="-5.8928E-09" iyy="2.953E-07" iyz="-4.2271E-10" izz="7.6154E-08" />
+		</inertial>
+		<visual>
+			<origin xyz="0 0 0" rpy="0 0 0" />
+			<geometry>
+				<mesh filename="package://abot_description/meshes/ir_f.STL" />
+			</geometry>
+			<material name="Yellow" />
+		</visual>
+		<collision>
+			<origin xyz="0 0 0" rpy="0 0 0" />
+			<geometry>
+				<mesh filename="package://abot_description/meshes/ir_f.STL" />
+			</geometry>
+		</collision>
+	</link>
+	<!-- IR sensor front joint -->
 	<joint name="ir_f_to_base" type="fixed">
-		<origin xyz="0.088 0 0.065" rpy="0 0 0" />
-		<parent link="base_link" />
+		<origin xyz="0.0874500000000004 0 0.031499999999999" rpy="0 0 0" />
+		<parent link="abot_base" />
 		<child link="ir_f" />
 		<axis xyz="0 0 0" />
 	</joint>
+	<!-- IR sensor left CAD link -->
+	<link name="ir_l">
+		<inertial>
+			<origin xyz="-0.0073719 -0.00051001 0.00027926" rpy="0 0 0" />
+			<mass value="0.0029707" />
+			<inertia ixx="3.1673E-07" ixy="6.7636E-10" ixz="-5.8928E-09" iyy="2.953E-07" iyz="-4.2271E-10" izz="7.6154E-08" />
+		</inertial>
+		<visual>
+			<origin xyz="0 0 0" rpy="0 0 0" />
+			<geometry>
+				<mesh filename="package://abot_description/meshes/ir_l.STL" />
+			</geometry>
+			<material name="Yellow" />
+		</visual>
+		<collision>
+			<origin xyz="0 0 0" rpy="0 0 0" />
+			<geometry>
+				<mesh filename="package://abot_description/meshes/ir_l.STL" />
+			</geometry>
+		</collision>
+	</link>
+	<!-- IR sensor left joint -->
+	<joint name="ir_l_to_base" type="fixed">
+		<origin xyz="-0.00999999999999981 0.0974499999999997 0.0315000000000011" rpy="0 0 1.57079632679489" />
+		<parent link="abot_base" />
+		<child link="ir_l" />
+		<axis xyz="0 0 0" />
+	</joint>
+	<!-- IR sensor right CAD link -->
+	<link name="ir_r">
+		<inertial>
+			<origin xyz="-0.0073719 0.00051001 -0.00027926" rpy="0 0 0" />
+			<mass value="0.0029707" />
+			<inertia ixx="3.1673E-07" ixy="-6.7636E-10" ixz="5.8928E-09" iyy="2.953E-07" iyz="-4.2271E-10" izz="7.6154E-08" />
+		</inertial>
+		<visual>
+			<origin xyz="0 0 0" rpy="0 0 0" />
+			<geometry>
+				<mesh filename="package://abot_description/meshes/ir_r.STL" />
+			</geometry>
+			<material name="Yellow" />
+		</visual>
+		<collision>
+			<origin xyz="0 0 0" rpy="0 0 0" />
+			<geometry>
+				<mesh filename="package://abot_description/meshes/ir_r.STL" />
+			</geometry>
+		</collision>
+	</link>
+	<!-- IR sensor right joint -->
+	<joint name="ir_r_to_base" type="fixed">
+		<origin xyz="-0.00999999999999882 -0.0974500000000003 0.0314999999999991" rpy="-3.14159265358979 0 -1.57079632679489" />
+		<parent link="abot_base" />
+		<child link="ir_r" />
+		<axis xyz="0 0 0" />
+	</joint>
+	<!-- IR sensor back CAD link -->
+	<link name="ir_b">
+		<inertial>
+			<origin xyz="-0.0073719 0.00051001 -0.00027926" rpy="0 0 0" />
+			<mass value="0.0029707" />
+			<inertia ixx="3.1673E-07" ixy="-6.7636E-10" ixz="5.8928E-09" iyy="2.953E-07" iyz="-4.2271E-10" izz="7.6154E-08" />
+		</inertial>
+		<visual>
+			<origin xyz="0 0 0" rpy="0 0 0" />
+			<geometry>
+				<mesh filename="package://abot_description/meshes/ir_b.STL" />
+			</geometry>
+			<material name="Yellow" />
+		</visual>
+		<collision>
+			<origin xyz="0 0 0" rpy="0 0 0" />
+			<geometry>
+				<mesh filename="package://abot_description/meshes/ir_b.STL" />
+			</geometry>
+		</collision>
+	</link>
+	<!-- IR sensor back joint -->
+	<joint name="ir_b_to_base" type="fixed">
+		<origin xyz="-0.10745 0 0.0315000000000011" rpy="3.14159265358979 0 -3.14159265358979" />
+		<parent link="abot_base" />
+		<child link="ir_b" />
+		<axis xyz="0 0 0" />
+	</joint>
+	<!-- IR sensor front right CAD link -->
+	<link name="ir_fr">
+		<inertial>
+			<origin xyz="-0.0073719 0.00051001 -0.00027926" rpy="0 0 0" />
+			<mass value="0.0029707" />
+			<inertia ixx="3.1673E-07" ixy="-6.7636E-10" ixz="5.8928E-09" iyy="2.953E-07" iyz="-4.2271E-10" izz="7.6154E-08" />
+		</inertial>
+		<visual>
+			<origin xyz="0 0 0" rpy="0 0 0" />
+			<geometry>
+				<mesh filename="package://abot_description/meshes/ir_fr.STL" />
+			</geometry>
+			<material name="Yellow" />
+		</visual>
+		<collision>
+			<origin xyz="0 0 0" rpy="0 0 0" />
+			<geometry>
+				<mesh filename="package://abot_description/meshes/ir_fr.STL" />
+			</geometry>
+		</collision>
+	</link>
+	<!-- IR sensor front right joint -->
+	<joint name="ir_fr_to_base" type="fixed">
+		<origin xyz="0.0589075558266301 -0.0689075558266286 0.0314999999999986" rpy="0 0 -0.785398163397442" />
+		<parent link="abot_base" />
+		<child link="ir_fr" />
+		<axis xyz="0 0 0" />
+	</joint>
+	<!-- IR sensor back right CAD link -->
+	<link name="ir_br">
+		<inertial>
+			<origin xyz="-0.0073719 0.00051001 -0.00027926" rpy="0 0 0" />
+			<mass value="0.0029707" />
+			<inertia ixx="3.1673E-07" ixy="-6.7636E-10" ixz="5.8928E-09" iyy="2.953E-07" iyz="-4.2271E-10" izz="7.6154E-08" />
+		</inertial>
+		<visual>
+			<origin xyz="0 0 0" rpy="0 0 0" />
+			<geometry>
+				<mesh filename="package://abot_description/meshes/ir_br.STL" />
+			</geometry>
+			<material name="Yellow" />
+		</visual>
+		<collision>
+			<origin xyz="0 0 0" rpy="0 0 0" />
+			<geometry>
+				<mesh filename="package://abot_description/meshes/ir_br.STL" />
+			</geometry>
+		</collision>
+	</link>
+	<!-- IR sensor back right joint -->
+	<joint name="ir_br_to_base" type="fixed">
+		<origin xyz="-0.0789075558266282 -0.0689075558266298 0.0315000000000001" rpy="-3.14159265358979 0 -2.35619449019234" />
+		<parent link="abot_base" />
+		<child link="ir_br" />
+		<axis xyz="0 0 0" />
+	</joint>
+	<!-- IR sensor back left CAD link -->
+	<link name="ir_bl">
+		<inertial>
+			<origin xyz="-0.0073719 0.00051001 -0.00027926" rpy="0 0 0" />
+			<mass value="0.0029707" />
+			<inertia ixx="3.1673E-07" ixy="-6.7636E-10" ixz="5.8928E-09" iyy="2.953E-07" iyz="-4.2271E-10" izz="7.6154E-08" />
+		</inertial>
+		<visual>
+			<origin xyz="0 0 0" rpy="0 0 0" />
+			<geometry>
+				<mesh filename="package://abot_description/meshes/ir_bl.STL" />
+			</geometry>
+			<material name="Yellow" />
+		</visual>
+		<collision>
+			<origin xyz="0 0 0" rpy="0 0 0" />
+			<geometry>
+				<mesh filename="package://abot_description/meshes/ir_bl.STL" />
+			</geometry>
+		</collision>
+	</link>
+	<!-- IR sensor back left joint -->
+	<joint name="ir_bl_to_base" type="fixed">
+		<origin xyz="-0.078908 0.068908 0.0315" rpy="-3.1416 0 2.3562" />
+		<parent link="abot_base" />
+		<child link="ir_bl" />
+		<axis xyz="0 0 0" />
+	</joint>
 	<!-- IR sensor front left CAD link -->
-	<link name="ir_l">
-		<inertial>
-			<origin xyz="-0.00737194484411242 0.000279264844105703 0.000510014496335439" rpy="0 0 0" />
-			<mass value="0.00297067826138337" />
-			<inertia ixx="3.16734695808955E-07" ixy="-5.89288167867935E-09" ixz="-6.76347714169545E-10" iyy="7.61538286810033E-08" iyz="4.22675785570517E-10" izz="2.95301261269084E-07" />
+	<link name="ir_fl">
+		<inertial>
+			<origin xyz="-0.0073719 0.00051001 -0.00027926" rpy="0 0 0" />
+			<mass value="0.0029707" />
+			<inertia ixx="3.1673E-07" ixy="-6.7636E-10" ixz="5.8928E-09" iyy="2.953E-07" iyz="-4.2271E-10" izz="7.6154E-08" />
 		</inertial>
 		<visual>
@@ -80,36 +248,8 @@
 	</link>
 	<!-- IR sensor front left joint -->
-	<joint name="ir_l_to_base" type="fixed">
-		<origin xyz="0 0.098 0.065" rpy="0 0 1.57" />
-		<parent link="base_link" />
-		<child link="ir_l" />
-		<axis xyz="0 0 0" />
-	</joint>
-	<!-- IR sensor front right CAD link -->
-	<link name="ir_r">
-		<inertial>
-			<origin xyz="-0.0073719435479474 0.000279266429044269 0.000510012687927432" rpy="0 0 0" />
-			<mass value="0.00297067925092848" />
-			<inertia ixx="3.16734825741921E-07" ixy="-5.89285028889523E-09" ixz="-6.76367534098839E-10" iyy="7.61538418054215E-08" iyz="4.2267880693731E-10" izz="2.95301389790314E-07" />
-		</inertial>
-		<visual>
-			<origin xyz="0 0 0" rpy="0 0 0" />
-			<geometry>
-				<mesh filename="package://abot_description/meshes/ir_fr.STL" />
-			</geometry>
-			<material name="Yellow" />
-		</visual>
-		<collision>
-			<origin xyz="0 0 0" rpy="0 0 0" />
-			<geometry>
-				<mesh filename="package://abot_description/meshes/ir_fr.STL" />
-			</geometry>
-		</collision>
-	</link>
-	<!-- IR sensor front right joint -->
-	<joint name="ir_r_to_base" type="fixed">
-		<origin xyz="0 -0.098 0.065" rpy="0 0 -1.57" />
-		<parent link="base_link" />
-		<child link="ir_r" />
+	<joint name="ir_fl_to_base" type="fixed">
+		<origin xyz="0.0589075558266294 0.0689075558266288 0.0315000000000001" rpy="0 0 0.785398163397444" />
+		<parent link="abot_base" />
+		<child link="ir_fl" />
 		<axis xyz="0 0 0" />
 	</joint>
