Commit message: 29.10.2020

File: ros/src/abot_description/urdf/abot.xacro (robot description, xacro)
@@ -4,6 +4,6 @@
 	<!-- Matherials -->
 	<xacro:include filename="$(find abot_description)/urdf/abot_matherials.xacro" />
-	<!-- base_link -->
-	<link name="base_link">
+	<!-- abot_base -->
+	<link name="abot_base">
 	  <inertial>
 			<origin xyz="-0.02452 1.4288E-14 0.021229" rpy="0 0 0" />
@@ -25,4 +25,15 @@
 		</collision>
 	</link>
+    <!-- base_link -->
+	<link name="base_link">
+		<visual>
+			<origin xyz="0 0 0" rpy="0 0 0" />
+		</visual>
+	</link>
+	<joint name="base_link_to_abot_base" type="fixed">
+		<origin xyz="0 0 0" rpy="0 0 0" />
+		<parent link="base_link" />
+		<child link="abot_base" />
+	</joint>
     <!-- Wheels -->
 	<xacro:include filename="$(find abot_description)/urdf/abot_left_wheel.xacro" />

File: ros/src/abot_description/urdf/abot_caster_wheel.xacro (robot description, xacro)
@@ -25,5 +25,5 @@
 	<joint name="caster_wheel_to_base" type="fixed">
 		<origin xyz="-0.078 0 -0.011" rpy="0 0 0" />
-		<parent link="base_link" />
+		<parent link="abot_base" />
 		<child link="abot_caster_wheel" />
 		<axis xyz="0 0 0" />

File: ros/src/abot_description/urdf/abot_left_wheel.xacro (robot description, xacro)
@@ -25,5 +25,5 @@
 	<joint name="left_wheel_to_base" type="continuous">
 		<origin xyz="0 0.068 0.0145" rpy="0 0 0" />
-		<parent link="base_link" />
+		<parent link="abot_base" />
 		<child link="abot_left_wheel" />
 		<axis xyz="0 1 0" />

File: ros/src/abot_description/urdf/abot_right_wheel.xacro (robot description, xacro)
@@ -25,5 +25,5 @@
 	<joint name="right_wheel_to_base" type="continuous">
 		<origin xyz="0 -0.068 0.0145" rpy="0 0 0" />
-		<parent link="base_link" />
+		<parent link="abot_base" />
 		<child link="abot_right_wheel" />
 		<axis xyz="0 1 0" />

Commit message: 29.10.2020

File: ros/src/abot_description/urdf/abot.xacro (robot description, xacro)
@@ -29,4 +29,7 @@
 		<visual>
 			<origin xyz="0 0 0" rpy="0 0 0" />
+            <geometry>
+				<sphere radius="0.001" />
+			</geometry>
 		</visual>
 	</link>

Commit message: 29.10.2020

File: ros/src/abot_description/urdf/abot.xacro (robot description, xacro)
@@ -2,4 +2,5 @@
 <robot name="abot"
 	xmlns:xacro="http://www.ros.org/wiki/xacro">
+	<xacro:property name="clearance" value="0.018" />
 	<!-- Matherials -->
 	<xacro:include filename="$(find abot_description)/urdf/abot_matherials.xacro" />
@@ -14,5 +15,5 @@
 			<origin xyz="0 0 0" rpy="0 0 0" />
 			<geometry>
-				<mesh filename="package://abot_description/meshes/base_link.STL" />
+				<mesh filename="package://abot_description/meshes/abot_base.STL" />
 			</geometry>
 			<material name="White" />
@@ -21,5 +22,5 @@
 			<origin xyz="0 0 0" rpy="0 0 0" />
 			<geometry>
-				<mesh filename="package://abot_description/meshes/base_link.STL" />
+				<mesh filename="package://abot_description/meshes/abot_base.STL" />
 			</geometry>
 		</collision>
@@ -39,4 +40,19 @@
 		<child link="abot_base" />
 	</joint>
+	<!-- base_footprint -->
+	<link name="base_footprint">
+		<visual>
+			<origin xyz="0 0 0" rpy="0 0 0" />
+			<geometry>
+				<cylinder length="0.001" radius="0.100" />
+			</geometry>
+			<material name="Blue" />
+		</visual>
+	</link>
+	<joint name="base_footprint_to_base_link" type="fixed">
+		<origin xyz="0 0 ${clearance}" rpy="0 0 0" />
+		<parent link="base_footprint" />
+		<child link="base_link" />
+	</joint>
     <!-- Wheels -->
 	<xacro:include filename="$(find abot_description)/urdf/abot_left_wheel.xacro" />

Commit message: 01.11.2020

File: ros/src/abot_description/urdf/abot.xacro (robot description, xacro)
@@ -7,8 +7,8 @@
 	<!-- abot_base -->
 	<link name="abot_base">
-	  <inertial>
-			<origin xyz="-0.02452 1.4288E-14 0.021229" rpy="0 0 0" />
-			<mass value="0.26675" />
-			<inertia ixx="0.00032378" ixy="-1.1141E-12" ixz="-9.1302E-06" iyy="0.00030073" iyz="-3.3253E-10" izz="0.000561" />
+		<inertial>
+  			<origin xyz="-0.018609547232146 0.00100725867922426 0.0368403920902579" rpy="0 0 0" />
+  			<mass value="0.38366067400424" />
+  			<inertia ixx="0.000455060033055237" ixy="-1.42665016686539E-06" ixz="-9.36574661563202E-06" iyy="0.000428067922539319" iyz="-4.00231856414886E-07" izz="0.000800906575951907" />
 		</inertial>
 		<visual>

Commit message: 02.11.2020

File: ros/src/abot_description/urdf/abot.xacro (robot description, xacro)
@@ -3,4 +3,6 @@
 	xmlns:xacro="http://www.ros.org/wiki/xacro">
 	<xacro:property name="clearance" value="0.018" />
+	<xacro:property name="wheel_radius" value="0.03195"/>
+	<xacro:property name="wheel_separation" value="0.128"/>
 	<!-- Matherials -->
 	<xacro:include filename="$(find abot_description)/urdf/abot_matherials.xacro" />

Commit message: 03.11.2020

File: ros/src/abot_description/urdf/abot.xacro (robot description, xacro)
@@ -5,4 +5,6 @@
 	<xacro:property name="wheel_radius" value="0.03195"/>
 	<xacro:property name="wheel_separation" value="0.128"/>
+	<xacro:property name="wheel_width" value="0.026"/>
+	<xacro:property name="PI" value="3.1415926"/>
 	<!-- Matherials -->
 	<xacro:include filename="$(find abot_description)/urdf/abot_matherials.xacro" />

File: ros/src/abot_description/urdf/abot_left_wheel.xacro (robot description, xacro)
@@ -23,8 +23,29 @@
 		</collision>
 	</link>
+	<!-- left_wheel_geometry -->
+	<link name="left_wheel">
+		<visual>
+			<origin xyz="0 0 0" rpy="${PI/2} 0 0" />
+			<geometry>
+				<cylinder length="${wheel_width}" radius="${wheel_radius}"/>
+			</geometry>
+			<material name="Green" />
+		</visual>
+		<collision>
+			<origin xyz="0 0 0" rpy="${PI/2} 0 0" />
+			<geometry>
+				<cylinder length="${wheel_width}" radius="${wheel_radius}"/>
+			</geometry>
+		</collision>
+	</link>
+	<joint name="left_wheel_to_abot_left_wheel" type="fixed">
+		<origin xyz="0 0 0" rpy="0 0 0" />
+		<parent link="left_wheel" />
+		<child link="abot_left_wheel" />
+	</joint>
 	<joint name="left_wheel_to_base" type="continuous">
 		<origin xyz="0 0.068 0.0145" rpy="0 0 0" />
 		<parent link="abot_base" />
-		<child link="abot_left_wheel" />
+		<child link="left_wheel" />
 		<axis xyz="0 1 0" />
 	</joint>

File: ros/src/abot_description/urdf/abot_right_wheel.xacro (robot description, xacro)
@@ -23,8 +23,28 @@
 		</collision>
 	</link>
+	<link name="right_wheel">
+		<visual>
+			<origin xyz="0 0 0" rpy="${PI/2} 0 0" />
+			<geometry>
+				<cylinder length="${wheel_width}" radius="${wheel_radius}"/>
+			</geometry>
+			<material name="Green" />
+		</visual>
+		<collision>
+			<origin xyz="0 0 0" rpy="${PI/2} 0 0" />
+			<geometry>
+				<cylinder length="${wheel_width}" radius="${wheel_radius}"/>
+			</geometry>
+		</collision>
+	</link>
+	<joint name="right_wheel_to_abot_right_wheel" type="fixed">
+		<origin xyz="0 0 0" rpy="0 0 0" />
+		<parent link="right_wheel" />
+		<child link="abot_right_wheel" />
+	</joint>
 	<joint name="right_wheel_to_base" type="continuous">
 		<origin xyz="0 -0.068 0.0145" rpy="0 0 0" />
 		<parent link="abot_base" />
-		<child link="abot_right_wheel" />
+		<child link="right_wheel" />
 		<axis xyz="0 1 0" />
 	</joint>
